File: PCB/PowerDistributionBoard.kicad_sch (KiCad schematic)
At the start: 61 parts, among them J1 Conn_01x02_Pin, J2 Conn_01x02_Socket, J3 Conn_01x02_Socket, J4 Conn_01x16_Socket, Q1 BSC026N08NS5, Q2 BSC026N08NS5, Q3 BSC026N08NS5, Q4 BSC026N08NS5, Q5 BSC026N08NS5, Q6 BSC026N08NS5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

Commit message: added firmware for controller, which is just a modified joystick example as of right now. There will need to be sone refactoring of this project to better reflect the electrical architecture at some point.
Parts:
- removed A1: RaspberryPi_Pico, Module:RaspberryPi_Pico_Common_Unspecified, symbol MCU_Module:RaspberryPi_Pico
- removed C1: 100n, symbol Device:C
- removed D1: D_Schottky, symbol Device:D_Schottky
- removed Q1, Q4, Q5, Q6: BSC026N08NS5, Package_TO_SOT_SMD:TDSON-8-1, symbol Transistor_FET:BSC026N08NS5
- removed R10, R11, R5, R6, R7, R8, R9: 1k, Resistor_SMD:R_1206_3216Metric, symbol Device:R
- removed R12: R, symbol Device:R
- removed U2: BQ76925, symbol Misc_PMlib:BQ76925
- removed U3: TEC2-4812WI, Converter_DCDC:Converter_DCDC_TRACO_TEC2-12xxWI_24xxWI_48xxWI_THT, symbol Converter_DCDC:TEC2-4812WI
- added J5: Conn_01x02_Pin, Connector_AMASS:AMASS_XT90PW-M_1x02_P10.90mm_Horizontal, symbol Connector:Conn_01x02_Pin
- added R29, R30: 1k, Resistor_SMD:R_1206_3216Metric, symbol Device:R
- added U2: UCC27524D, Package_SO:SOIC-8_3.9x4.9mm_P1.27mm, symbol Driver_FET:UCC27524D
- R3, R4: value 1k -> R; footprint Resistor_SMD:R_1206_3216Metric -> (none)
Connections:
- net V_{IN}: now also R29.1, R30.1; no longer Q2.5 (D), Q3.5 (D), R3.1
- net V_{OUT}: now also R29.2, R30.2; no longer Q2.1 (S), Q2.2 (S), Q2.3 (S), Q3.1 (S), Q3.2 (S), Q3.3 (S)
- net at R3.2: now also Q3.4 (G); no longer R4.1
- net at R4.2: now also Q2.4 (G)
- net at U1.1 (ENA), U1.4 (INB): no longer U1.6 (V_{DD})
- new net: R3.1, U2.7 (OUTA)
- new net: Q3.1 (S), Q3.2 (S), Q3.3 (S)
- new net: Q2.1 (S), Q2.2 (S), Q2.3 (S), Q3.5 (D), U2.3 (GND)
- new net: R4.1, U2.5 (OUTB)
- now unconnected: R2.1
Other:
- moved on the sheet: C10, C11, C12, C13, C14, C15, C16, C2, C3, C4, C5, C6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
